File: KiCad Files/rev1c/rev1c.kicad_pcb (KiCad board)
At the start: 2 copper layers, 285 x 94.6 mm, 158 parts, among them SW1 SW_Push, SW10 SW_Push, SW11 SW_Push, SW12 SW_Push, SW13 SW_Push, SW14 SW_Push, SW15 SW_Push, SW16 SW_Push, SW17 SW_Push, SW18 SW_Push, SW19 SW_Push, SW2 SW_Push, SW20 SW_Push, SW21 SW_Push, SW22 SW_Push, SW23 SW_Push, SW24 SW_Push, SW25 SW_Push, SW26 SW_Push, SW27 SW_Push, SW28 SW_Push, SW29 SW_Push, SW3 SW_Push, SW30 SW_Push, SW31 SW_Push, SW32 SW_Push, SW33 SW_Push, SW34 SW_Push, SW35 SW_Push, SW36 SW_Push, SW37 SW_Push, SW38 SW_Push, SW39 SW_Push, SW4 SW_Push, SW40 SW_Push, SW41 SW_Push, SW42 SW_Push, SW43 SW_Push, SW44 SW_Push, SW45 SW_Push, SW46 SW_Push, SW47 SW_Push, SW48 SW_Push, SW49 SW_Push, SW5 SW_Push, SW50 SW_Push, SW51 SW_Push, SW52 SW_Push, SW53 SW_Push, SW54 SW_Push, SW55 SW_Push, SW56 SW_Push, SW57 SW_Push, SW58 SW_Push, SW59 SW_Push, SW6 SW_Push, SW60 SW_Push, SW63 SW_Push, SW65 SW_Push, SW66 SW_Push, SW67 SW_Push, SW68 SW_Push, SW7 SW_Push, SW8 SW_Push, SW9 SW_Push

Commit message: Rev1c preliminarty update
Changes to Schematic:
- Added switches to support different layouts
- Added One BAV70 to support said switches

Changes to PCB:
- Imported changes from schematic, placed some of the switches but needs more work
Parts:
- added D31: BAV70, PCM_Package_TO_SOT_SMD_AKL:SOT-23, F.Cu at (218.1, 197.0)
- added SW61: SW_Push, PCM_Switch_Keyboard_Hotswap_Kailh:SW_Hotswap_Kailh_MX_Plated_2.75u, F.Cu at (193.3, 176.5)
- added SW62: SW_Push, PCM_Switch_Keyboard_Hotswap_Kailh:SW_Hotswap_Kailh_MX_Plated_2.25u, F.Cu at (264.7, 176.5)
- added SW64: SW_Push, PCM_Switch_Keyboard_Hotswap_Kailh:SW_Hotswap_Kailh_MX_Plated_1.00u, F.Cu at (393.1, 67.3)
- added SW69: SW_Push, PCM_Switch_Keyboard_Hotswap_Kailh:SW_Hotswap_Kailh_MX_Plated_1.00u, F.Cu at (371.7, 67.3)
- added SW70: SW_Push, PCM_Switch_Keyboard_Hotswap_Kailh:SW_Hotswap_Kailh_MX_Plated_1.50u, F.Cu at (412.0, 114.6)
- added SW71: SW_Push, PCM_Switch_Keyboard_Hotswap_Kailh:SW_Hotswap_Kailh_MX_Plated_2.25u, F.Cu at (405.2, 133.7)
- added SW72: SW_Push, PCM_Switch_Keyboard_Hotswap_Kailh:SW_Hotswap_Kailh_MX_Plated_1.25u, F.Cu at (231.4, 176.5)
Connections:
- D21 pad 1: unconnected-(D21-A-Pad1) -> Net-(D21-A-Pad1)
- SW28 pad 2: Net-(D14-A-Pad2) -> Net-(D21-A-Pad1)
- SW63 pad 2: Net-(D30-A-Pad2) -> Net-(D31-A-Pad1)
Routing:
- removed copper zone on B.Cu, net GND
- removed copper zone on F.Cu, net GND

Commit message: update on pcb
Parts:
- removed SW70: SW_Push, PCM_Switch_Keyboard_Hotswap_Kailh:SW_Hotswap_Kailh_MX_Plated_1.50u
- removed SW71: SW_Push, PCM_Switch_Keyboard_Hotswap_Kailh:SW_Hotswap_Kailh_MX_Plated_2.25u
- D31: moved to B.Cu
- moved SW64 39.3 mm to (371.9, 100.3), turned to 180 degrees
- moved SW69 38.0 mm to (352.8, 100.3), turned to 180 degrees
- moved D31 36.2 mm to (249.5, 178.9), turned to -90 degrees
- turned ? to 90 degrees
Routing:
- net Net-(LED8-DOUT): track 62.4 -> 14.4 mm
- net +5V: track 606.3 -> 558.6 mm
- net Net-(D31-A-Pad1): track 0.00 -> 22.2 mm
- net Net-(D31-A-Pad2): track 0.00 -> 22.2 mm
- net Col4: track 126.1 -> 148.1 mm
- net Col8: track 200.8 -> 220.8 mm
- net Col6: track 183.5 -> 195.1 mm
- net Col13: track 314.5 -> 304.4 mm
Other:
- board text added: "Slothie60 Rev. 1c"
- board text removed: "Slothie60 Rev. 1b"

Commit message: Updates
Parts:
- added REF**: Stabilizer_Cherry_MX_2.00u, PCM_Mounting_Keyboard_Stabilizer:Stabilizer_Cherry_MX_2.00u, F.Cu at (264.7, 176.5)
- added REF**: Stabilizer_Cherry_MX_2.00u, PCM_Mounting_Keyboard_Stabilizer:Stabilizer_Cherry_MX_2.00u, F.Cu at (217.1, 176.5)
- SW61: footprint PCM_Switch_Keyboard_Hotswap_Kailh:SW_Hotswap_Kailh_MX_Plated_2.75u -> PCM_Switch_Keyboard_Hotswap_Kailh:SW_Hotswap_Kailh_MX_Plated_1.25u
- SW72: footprint PCM_Switch_Keyboard_Hotswap_Kailh:SW_Hotswap_Kailh_MX_Plated_1.25u -> PCM_Switch_Keyboard_Hotswap_Kailh:SW_Hotswap_Kailh_MX_Plated_2.75u
- moved SW61 14.3 mm to (179.0, 176.5)
- moved SW72 14.3 mm to (217.1, 176.5)
- moved LED12 4.54 mm to (260.7, 165.7)
- moved C12 4.54 mm to (256.1, 166.5)
- moved LED8 2.06 mm to (364.7, 110.7)
- moved C8 2.03 mm to (369.5, 109.9)
- turned ? to -90 degrees
Connections:
- SW72 pad 1: Net-(D31-A-Pad1) -> Col6
- SW72 pad 2: Col6 -> Net-(D31-A-Pad1)
Routing:
- net +5V: track 558.6 -> 613.8 mm
- net Net-(D21-A-Pad1): track 0.00 -> 48.9 mm
- net Net-(LED8-DOUT): track 14.4 -> 60.9 mm
- net Col13: track 304.4 -> 329.7 mm
- net Net-(D7-A-Pad2): track 26.4 -> 49.0 mm
- net Net-(D31-A-Pad1): track 22.2 -> 43.0 mm
- net Net-(D14-A-Pad2): track 38.6 -> 49.0 mm
- net GND: track 48.8 -> 56.7 mm
- net Net-(LED12-DOUT): track 31.8 -> 36.3 mm
- net Net-(LED11-DOUT): track 31.8 -> 27.3 mm
- net Col6: track 195.1 -> 190.7 mm
- net Net-(LED7-DOUT): track 32.4 -> 34.4 mm
- net Row4: track 291.7 -> 293.7 mm
