File: KiCad Files/rev1c/rev1c.kicad_pcb (KiCad board)
At the start: 2 copper layers, 285 x 94.6 mm, 166 parts, among them SW1 SW_Push, SW10 SW_Push, SW11 SW_Push, SW12 SW_Push, SW13 SW_Push, SW14 SW_Push, SW15 SW_Push, SW16 SW_Push, SW17 SW_Push, SW18 SW_Push, SW19 SW_Push, SW2 SW_Push, SW20 SW_Push, SW21 SW_Push, SW22 SW_Push, SW23 SW_Push, SW24 SW_Push, SW25 SW_Push, SW26 SW_Push, SW27 SW_Push, SW28 SW_Push, SW29 SW_Push, SW3 SW_Push, SW30 SW_Push, SW31 SW_Push, SW32 SW_Push, SW33 SW_Push, SW34 SW_Push, SW35 SW_Push, SW36 SW_Push, SW37 SW_Push, SW38 SW_Push, SW39 SW_Push, SW4 SW_Push, SW40 SW_Push, SW41 SW_Push, SW42 SW_Push, SW43 SW_Push, SW44 SW_Push, SW45 SW_Push, SW46 SW_Push, SW47 SW_Push, SW48 SW_Push, SW49 SW_Push, SW5 SW_Push, SW50 SW_Push, SW51 SW_Push, SW52 SW_Push, SW53 SW_Push, SW54 SW_Push, SW55 SW_Push, SW56 SW_Push, SW57 SW_Push, SW58 SW_Push, SW59 SW_Push, SW6 SW_Push, SW60 SW_Push, SW61 SW_Push, SW62 SW_Push, SW63 SW_Push, SW64 SW_Push, SW65 SW_Push, SW66 SW_Push, SW67 SW_Push, SW68 SW_Push, SW69 SW_Push, SW7 SW_Push, SW72 SW_Push, SW8 SW_Push, SW9 SW_Push

Commit message: Plate stuff
- Added a plate design for rev 1b
- Some updates to 1c
Parts:
- moved ? 5.05 mm to (239.8, 174.0)
Routing:
- net Net-(D30-A-Pad2): track 69.2 -> 21.6 mm
- net Col13: track 329.7 -> 334.8 mm
- net Net-(LED7-DOUT): track 34.4 -> 31.5 mm
- net Net-(LED8-DOUT): track 60.9 -> 63.7 mm
- net +5V: track 613.8 -> 612.5 mm
- added copper zone on B.Cu, net GND
- added copper zone on F.Cu, net GND
Other:
- board text added: "1.25U"
- board text added: "2.25U"
- board text added: "SLOTHIE"
