File: KiCad Files/rev2a/KeyMatrix.kicad_sch (KiCad schematic)
At the start: 103 parts, among them SW1 SW_Push, SW10 SW_Push, SW11 SW_Push, SW12 SW_Push, SW13 SW_Push, SW14 SW_Push, SW15 SW_Push, SW16 SW_Push, SW17 SW_Push, SW18 SW_Push, SW19 SW_Push, SW2 SW_Push, SW20 SW_Push, SW21 SW_Push, SW22 SW_Push, SW23 SW_Push, SW24 SW_Push, SW25 SW_Push, SW26 SW_Push, SW27 SW_Push, SW28 SW_Push, SW29 SW_Push, SW3 SW_Push, SW30 SW_Push, SW31 SW_Push, SW32 SW_Push, SW33 SW_Push, SW34 SW_Push, SW35 SW_Push, SW36 SW_Push, SW37 SW_Push, SW38 SW_Push, SW39 SW_Push, SW4 SW_Push, SW40 SW_Push, SW41 SW_Push, SW42 SW_Push, SW43 SW_Push, SW44 SW_Push, SW45 SW_Push, SW46 SW_Push, SW47 SW_Push, SW48 SW_Push, SW49 SW_Push, SW5 SW_Push, SW50 SW_Push, SW51 SW_Push, SW52 SW_Push, SW53 SW_Push, SW54 SW_Push, SW55 SW_Push, SW56 SW_Push, SW57 SW_Push, SW58 SW_Push, SW59 SW_Push, SW6 SW_Push, SW60 SW_Push, SW61 SW_Push, SW62 SW_Push, SW63 SW_Push, SW64 SW_Push, SW65 SW_Push, SW66 SW_Push, SW67 SW_Push, SW68 SW_Push, SW69 SW_Push, SW7 SW_Push, SW72 SW_Push, SW8 SW_Push, SW9 SW_Push

Commit message: rev2a
- basic layout
- leds
- rp2040 with all necessary things
Parts:
- removed SW29: SW_Push, PCM_Switch_Keyboard_Hotswap_Kailh:SW_Hotswap_Kailh_MX_Plated_1.25u, symbol Switch:SW_Push_45deg
- removed SW55: SW_Push, PCM_Switch_Keyboard_Hotswap_Kailh:SW_Hotswap_Kailh_MX_Plated_1.75u, symbol Switch:SW_Push_45deg
- removed SW57, SW64, SW69: SW_Push, PCM_Switch_Keyboard_Hotswap_Kailh:SW_Hotswap_Kailh_MX_Plated_1.00u, symbol Switch:SW_Push_45deg
- removed SW62: SW_Push, PCM_Switch_Keyboard_Hotswap_Kailh:SW_Hotswap_Kailh_MX_Plated_2.25u, symbol Switch:SW_Push_45deg
- removed SW72: SW_Push, PCM_Switch_Keyboard_Hotswap_Kailh:SW_Hotswap_Kailh_MX_Plated_2.75u, symbol Switch:SW_Push_45deg
- added SW58: SW_Push, PCM_Switch_Keyboard_Hotswap_Kailh:SW_Hotswap_Kailh_MX_Plated_2.75u, symbol Switch:SW_Push_45deg
- added SW60: SW_Push, PCM_Switch_Keyboard_Hotswap_Kailh:SW_Hotswap_Kailh_MX_Plated_1.25u, symbol Switch:SW_Push_45deg
- SW61: footprint PCM_Switch_Keyboard_Hotswap_Kailh:SW_Hotswap_Kailh_MX_Plated_1.25u -> PCM_Switch_Keyboard_Hotswap_Kailh:SW_Hotswap_Kailh_MX_Plated_2.25u
- renumbered SW30 to SW29, SW31 to SW30, SW32 to SW31, SW33 to SW32, SW34 to SW33, SW35 to SW34, SW36 to SW35, SW37 to SW36, SW38 to SW37, SW39 to SW38, SW40 to SW39, SW41 to SW40, SW42 to SW41, SW43 to SW42, SW44 to SW43, SW45 to SW44, SW46 to SW45, SW47 to SW46, SW48 to SW47, SW49 to SW48, SW50 to SW49, SW51 to SW50, SW52 to SW51, SW53 to SW52, SW54 to SW53, SW56 to SW54, SW58 to SW55, SW59 to SW56, SW60 to SW57, SW63 to SW59, SW65 to SW62, SW66 to SW63, SW67 to SW64, SW68 to SW65
Connections:
- net Col0: now also SW1.2; no longer SW1.1
- net Col1: now also SW2.2; no longer SW2.1
- net Col4: now also SW58.1; no longer SW61.1
- net Col6: now also SW60.2
- net Col8: now also SW61.1
- net at D1.2 (A): now also SW2.1; no longer SW2.2
- net at SW55.2: now also D29.2 (A); no longer D29.1 (A)
- net at SW54.2: now also D28.2 (A); no longer D28.1 (A)
- net at D9.1 (A): now also SW18.2; no longer SW17.2
- net at D9.2 (A): now also SW17.2; no longer SW18.2
- net at D10.1 (A): now also SW20.2; no longer SW19.2
- net at D10.2 (A): now also SW19.2; no longer SW20.2
- net at SW56.2: now also D29.1 (A); no longer D29.2 (A)
- net at SW62.2: now also D32.2 (A); no longer D32.1 (A)
- net at D12.1 (A): now also SW24.2; no longer SW23.2
- net at D12.2 (A): now also SW23.2; no longer SW24.2
- net at D31.2 (A): now also SW59.2, SW60.1
- net at D13.1 (A): now also SW26.2; no longer SW25.2
- net at D13.2 (A): now also SW25.2; no longer SW26.2
- net at D30.1 (A): now also SW58.2; no longer SW57.2
- net at D30.2 (A): now also SW57.2; no longer SW61.2
- net at SW21.2: now also D11.2 (A); no longer D11.1 (A)
- net at D14.1 (A): now also SW28.2; no longer SW27.2
- net at D14.2 (A): now also SW27.2
- net at D1.1 (A): now also SW1.1; no longer SW1.2
- net at SW22.2: now also D11.1 (A); no longer D11.2 (A)
- net at D33.1 (A): now also SW65.2; no longer SW64.2
- net at D33.2 (A): now also SW64.2; no longer SW65.2
- net at SW16.2: now also D8.1 (A); no longer D8.2 (A)
- net at D21.1 (A): no longer SW28.2
- net at SW63.2: now also D32.1 (A); no longer D32.2 (A)
- net at D31.1 (A): now also SW61.2; no longer SW59.2
- net at SW15.2: now also D8.2 (A); no longer D8.1 (A)
- no-connect marks 0 -> 2
Other:
- note removed: "Caps 1.25/1.75U"
- moved on the sheet: SW28
